File: card-b-logic.sch (KiCad schematic (older format))
At the start: 23 parts

Commit message: Adds PDF of all the pages
Connections:
- net at G?.~ (X): now also G?.~ (X), G?.~ (X); no longer G?.~
- new net: G?.~, G?.~ (X) (x5)
- new net: G?.~, G?.~ (R), G?.~ (X)
- new net: G?.~, G?.~ (S)
- new net: G?.~ (R), G?.~ (X), G?.~ (X) (x2)
- new net: G?.~ (X), G?.~ (X)
- new net: G?.~ (S), G?.~ (X) (x2)
Changed lines of the file:
@@
 EESchema Schematic File Version 2
+LIBS:Friden-130-rescue
 LIBS:power
 LIBS:device
@@
 77 A7 A8 A8 88 D3 A7 4F EB 0C 8F 17 2C 58 80 9F 9F 1F 75 75 75 9C 3C 79 72 D8 FD E2 27 83 BB 4A
 72 97 BB 0C C3 2F 33 7D C5 5D EE 32 81 88 81 3B DB 71 E6 2E 77 99 64 FE 1F 65 78 2F 4D AD 02 B8
-F6 00 00 00 00 49 45 4E 44 AE 42 60 82 6D
+F6 00 00 00 00 49 45 4E 44 AE 42 60 82 8C
 EndData
 $EndBitmap
