File: pwr.sch (KiCad schematic (older format))
At the start: 93 parts, among them Q1 2N669, Q2 2N669, Q3 2N669, Q4 2N669, Q5 2N1305, Q6 2N1305, Q7 2N1305, T1 FridenTransformer, T2 TRANSFO, U1 STABI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

Commit message: Adds PDF of all the pages
Parts:
- RV4, RV5: symbol POT -> POT-RESCUE-Friden-130
