File: slot3a.sch (KiCad schematic (older format))
At the start: 354 parts, among them Q1 2N2635, Q10 2N2635, Q11 2N1304, Q12 2N2635, Q13 2N1305, Q14 2N1305, Q15 2N2635, Q16 2N2635, Q17 2N2635, Q18 2N2635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

Commit message: Adds PDF of all the pages
Changed lines of the file:
@@
 EESchema Schematic File Version 2
+LIBS:Friden-130-rescue
 LIBS:power
 LIBS:device
@@
 	6600 11050 6650 11050
 Wire Wire Line
-	6650 10850 6650 11050
+	6650 11050 6650 10850
 Wire Wire Line
 	3000 10850 23000 10850
