File: slot4b-ckt.sch (KiCad schematic (older format))
At the start: 347 parts, among them Q1 2N2635, Q10 2N2635, Q11 2N1304, Q12 2N2635, Q13 2N1304, Q14 2N2635, Q15 2N2635, Q16 2N2635, Q17 2N1304, Q18 2N1305, Q19 2N2635, Q2 2N2635, Q20 2N1305, Q21 2N1304, Q22 2N1305, Q23 2N2635, Q24 2N1304, Q25 2N1304, Q26 2N1305, Q27 2N1305, Q28 2N1304, Q29 2N1305, Q3 2N2635, Q30 2N1305, Q31 2N1304, Q32 2N1305, Q33 2N1304, Q34 2N1305, Q35 2N1305, Q36 2N1305, Q37 2N1305, Q38 2N1305, Q39 2N1305, Q4 2N1304, Q40 2N1305, Q41 2N1305, Q42 2N1305, Q43 2N1305, Q44 2N1305, Q45 2N1305, Q46 2N1305, Q47 2N1305, Q48 2N1305, Q49 2N1305, Q5 2N2635, Q6 2N1304, Q7 2N2635, Q8 2N1304, Q9 2N2635

Commit message: Adds PDF of all the pages
Parts:
- VR1, VR2, VR3, VR4, VR5: symbol POT -> POT-RESCUE-Friden-130
Changed lines of the file:
@@
 EESchema Schematic File Version 2
+LIBS:Friden-130-rescue
 LIBS:power
 LIBS:device
@@
 $Descr A2 23386 16535
 encoding utf-8
-Sheet 10 25
+Sheet 11 25
 Title ""
 Date ""
@@
 $EndComp
 $Comp
-L POT VR1
+L POT-RESCUE-Friden-130 VR1
 U 1 1 57FCCEFF
 P 23350 -2450
+AR Path="/57FCCEFF" Ref="VR1"  Part="1"
+AR Path="/57D11156/57F81E9F/57FCCEFF" Ref="VR1"  Part="1"
 F 0 "VR1" H 23350 -2550 50  0000 C CNN
 F 1 "POT" H 23350 -2450 50  0000 C CNN
@@
 $EndComp
 $Comp
-L POT VR2
+L POT-RESCUE-Friden-130 VR2
 U 1 1 57FCD73D
 P 22750 -2400
+AR Path="/57FCD73D" Ref="VR2"  Part="1"
+AR Path="/57D11156/57F81E9F/57FCD73D" Ref="VR2"  Part="1"
 F 0 "VR2" H 22750 -2500 50  0000 C CNN
 F 1 "POT" H 22750 -2400 50  0000 C CNN
@@
 $EndComp
 $Comp
-L POT VR3
+L POT-RESCUE-Friden-130 VR3
 U 1 1 57FCDB6D
 P 22200 -2500
+AR Path="/57FCDB6D" Ref="VR3"  Part="1"
+AR Path="/57D11156/57F81E9F/57FCDB6D" Ref="VR3"  Part="1"
 F 0 "VR3" H 22200 -2600 50  0000 C CNN
 F 1 "POT" H 22200 -2500 50  0000 C CNN
@@
 $EndComp
 $Comp
-L POT VR4
+L POT-RESCUE-Friden-130 VR4
 U 1 1 57FCDFA6
 P 21700 -2350
+AR Path="/57FCDFA6" Ref="VR4"  Part="1"
+AR Path="/57D11156/57F81E9F/57FCDFA6" Ref="VR4"  Part="1"
 F 0 "VR4" H 21700 -2450 50  0000 C CNN
 F 1 "POT" H 21700 -2350 50  0000 C CNN
@@
 $EndComp
 $Comp
-L POT VR5
+L POT-RESCUE-Friden-130 VR5
 U 1 1 57FCE3E6
 P 21100 -2500
+AR Path="/57FCE3E6" Ref="VR5"  Part="1"
+AR Path="/57D11156/57F81E9F/57FCE3E6" Ref="VR5"  Part="1"
 F 0 "VR5" H 21100 -2600 50  0000 C CNN
 F 1 "POT" H 21100 -2500 50  0000 C CNN
