File: video.sch (KiCad schematic (older format))
At the start: 22 parts, among them Q1 2N2043, Q2 2N2043, Q3 2N2043, Q4 2N2043

Commit message: Adds PDF of all the pages
Parts:
- RV1, RV2, RV3: symbol POT -> POT-RESCUE-Friden-130
Changed lines of the file:
@@
 EESchema Schematic File Version 2
+LIBS:Friden-130-rescue
 LIBS:power
 LIBS:device
@@
 $Descr A4 11693 8268
 encoding utf-8
-Sheet 6 25
+Sheet 7 25
 Title "Video deflection board"
 Date "13 Aug 2016"
@@
 	4200 3650 4200 3800
 $Comp
-L POT RV1
+L POT-RESCUE-Friden-130 RV1
 U 1 1 57C3953E
 P 3850 2050
+AR Path="/57C3953E" Ref="RV1"  Part="1"
+AR Path="/57C38C95/57C3953E" Ref="RV1"  Part="1"
 F 0 "RV1" H 3850 1950 50  0000 C CNN
 F 1 "POT" H 3850 2050 50  0000 C CNN
@@
 ASTIG.
 $Comp
-L POT RV2
+L POT-RESCUE-Friden-130 RV2
 U 1 1 57C3A763
 P 5100 2300
+AR Path="/57C3A763" Ref="RV2"  Part="1"
+AR Path="/57C38C95/57C3A763" Ref="RV2"  Part="1"
 F 0 "RV2" H 5100 2200 50  0000 C CNN
 F 1 "POT" H 5100 2300 50  0000 C CNN
@@
 	6350 3000 7100 3000
 $Comp
-L POT RV3
+L POT-RESCUE-Friden-130 RV3
 U 1 1 57C3C7F8
 P 6500 2300
+AR Path="/57C3C7F8" Ref="RV3"  Part="1"
+AR Path="/57C38C95/57C3C7F8" Ref="RV3"  Part="1"
 F 0 "RV3" H 6500 2200 50  0000 C CNN
 F 1 "POT" H 6500 2300 50  0000 C CNN
@@
 77 A7 A8 A8 88 D3 A7 4F EB 0C 8F 17 2C 58 80 9F 9F 1F 75 75 75 9C 3C 79 72 D8 FD E2 27 83 BB 4A
 72 97 BB 0C C3 2F 33 7D C5 5D EE 32 81 88 81 3B DB 71 E6 2E 77 99 64 FE 1F 65 78 2F 4D AD 02 B8
-F6 00 00 00 00 49 45 4E 44 AE 42 60 82 6D
+F6 00 00 00 00 49 45 4E 44 AE 42 60 82 8C
 EndData
 $EndBitmap
